File: Moddlers_Arduino_Uno_Shield.kicad_pcb (KiCad board)
At the start: 2 copper layers, 68.6 x 53.3 mm, 6 parts, among them J1 POWER, J2 ANALOG, J3 DIGITAL-PWM, J4 DIGITAL-PWM, J5 ICSP

Commit message: Update to KiCAD Version 6
Other:
- net class Default removed
